Commit message: gps

File: ros2_ws/src/eddy_description/urdf/eddy.urdf.xacro (robot description, xacro)
@@ -58,5 +58,5 @@
   <link name="thruster_left_link">
   </link>
-  <joint name="thruster_left_joint" type="continuous">
+  <joint name="thruster_left_joint" type="fixed">
     <parent link="base_link"/>
     <child link="thruster_left_link"/>
@@ -67,5 +67,5 @@
   <link name="thruster_right_link">
   </link>
-  <joint name="thruster_right_joint" type="continuous">
+  <joint name="thruster_right_joint" type="fixed">
     <parent link="base_link"/>
     <child link="thruster_right_link"/>

File: ros2_ws/src/eddy_gazebo/urdf/eddy.gazebo.xacro (robot description, xacro)
@@ -23,5 +23,5 @@
       </ros>
       <command_topic>/$(arg robot_name)/cmd_vel</command_topic>
-      <odometryTopic>/$(arg robot_name)/odom</odometryTopic>
+      <odometryTopic>/$(arg robot_name)/odometry</odometryTopic>
       <robot_base_frame>$(arg robot_name)/base_footprint</robot_base_frame>
       <odometry_frame>$(arg robot_name)/odom</odometry_frame>
@@ -38,4 +38,5 @@
           <remapping>gps_controller/out:=gps</remapping>
         </ros>
+        <frame_name>$(arg robot_name)/base_footprint</frame_name>
       </plugin>
     </sensor>
@@ -55,4 +56,5 @@
           <remapping>~/out:=imu</remapping>
         </ros>
+        <frame_name>$(arg robot_name)/base_footprint</frame_name>
       </plugin>
     </sensor>
